Commit message: first commit

File: urdf/HEBI.urdf (robot description, URDF)
Before this commit: robot HEBI, 22 links, 21 joints
Links:
- removed link leg_fl_extension
- removed link leg_fl_fixed
- removed link leg_fl_pitch
- removed link leg_fl_roll
- removed link leg_fr_extension
- removed link leg_fr_fixed
- removed link leg_fr_pitch
- removed link leg_fr_roll
- removed link leg_rl_extension
- removed link leg_rl_fixed
- removed link leg_rl_pitch
- removed link leg_rl_roll
- removed link leg_rr_extension
- removed link leg_rr_fixed
- removed link leg_rr_pitch
- removed link leg_rr_roll
- removed link track_fl
- removed link track_fr
- removed link track_rl
- removed link track_rr
- link base_link: mass 10 -> None; geometry visual mesh filename=package://intro_robotics_labs/my_CAD/chassis-Body.stl scale=0.01 0.01 0.01
Joints:
- removed joint leg_fl_fixed_joint
- removed joint leg_fl_pitch_joint
- removed joint leg_fl_prismatic
- removed joint leg_fl_roll_joint
- removed joint leg_fl_track_joint
- removed joint leg_fr_fixed_joint
- removed joint leg_fr_pitch_joint
- removed joint leg_fr_prismatic
- removed joint leg_fr_roll_joint
- removed joint leg_fr_track_joint
- removed joint leg_rl_fixed_joint
- removed joint leg_rl_pitch_joint
- removed joint leg_rl_prismatic
- removed joint leg_rl_roll_joint
- removed joint leg_rl_track_joint
- removed joint leg_rr_fixed_joint
- removed joint leg_rr_pitch_joint
- removed joint leg_rr_prismatic
- removed joint leg_rr_roll_joint
- removed joint leg_rr_track_joint

Commit message: UPDATE package name

File: urdf/HEBI.urdf (robot description, URDF)
Before this commit: robot simple_robot, 2 links, 1 joints
Links:
- link base_link: geometry visual mesh filename=package://hebi_robot/my_CAD/chassis-Body.stl scale=0.01 0.01 0.01

File: urdf/test.urdf (robot description, URDF)
Before this commit: robot simple_robot, 6 links, 5 joints
Links:
- link base_link: geometry visual mesh filename=package://hebi_robot/my_CAD/chassis1.stl scale=0.01 0.01 0.01
- link lr_shoulder: geometry collision mesh filename=package://hebi_robot/my_CAD/wheel.stl scale=0.01 0.01 0.01; visual mesh filename=package://hebi_robot/my_CAD/wheel.stl scale=0.01 0.01 0.01

Commit message: hebi moves

File: urdf/HEBI.urdf (robot description, URDF)
Before this commit: robot simple_robot, 2 links, 1 joints
Links:
- added link lf_foot, mass 1.0; collision cylinder length=0.1 radius=0.015; visual cylinder length=0.1 radius=0.001
- added link lf_foot_mid, mass 1.0; collision cylinder length=0.025 radius=0.001; visual cylinder length=0.025 radius=0.001
- added link lf_foot_mid_2, mass 1.0; collision sphere radius=0.005; visual sphere radius=0.005
- added link lf_foot_r, mass 1.0; collision sphere radius=0.01; visual sphere radius=0.01
- added link lf_leg, mass 1.0; collision cylinder length=0.1 radius=0.01; visual cylinder length=0.1 radius=0.0125
- added link lf_leg_ext, mass 1.0; collision cylinder length=0.1 radius=0.01; visual cylinder length=0.1 radius=0.0075
- added link lf_shoulder, mass 0.5; collision mesh filename=package://intro_robotics_labs/my_CAD/shoulder.stl scale=0.01 0.01 0.01; visual mesh filename=package://intro_robotics_labs/my_CAD/shoulder.stl scale=0.01 0.01 0.01
- added link lf_wheel_front, mass 1.0; collision mesh filename=package://intro_robotics_labs/my_CAD/wheel.stl scale=0.001 0.001 0.001; visual mesh filename=package://intro_robotics_labs/my_CAD/wheel.stl scale=0.001 0.001 0.001
- added link lf_wheel_rear, mass 1.0; collision mesh filename=package://intro_robotics_labs/my_CAD/wheel.stl scale=0.001 0.001 0.001; visual mesh filename=package://intro_robotics_labs/my_CAD/wheel.stl scale=0.001 0.001 0.001
- added link lr_foot, mass 1.0; collision cylinder length=0.1 radius=0.015; visual cylinder length=0.1 radius=0.001
- added link lr_foot_mid, mass 1.0; collision cylinder length=0.025 radius=0.001; visual cylinder length=0.025 radius=0.001
- added link lr_foot_mid_2, mass 1.0; collision sphere radius=0.005; visual sphere radius=0.005
- added link lr_foot_r, mass 1.0; collision sphere radius=0.01; visual sphere radius=0.01
- added link lr_leg, mass 1.0; collision cylinder length=0.1 radius=0.01; visual cylinder length=0.1 radius=0.0125
- added link lr_leg_ext, mass 1.0; collision cylinder length=0.1 radius=0.01; visual cylinder length=0.1 radius=0.0075
- added link lr_shoulder, mass 0.5; collision mesh filename=package://intro_robotics_labs/my_CAD/shoulder.stl scale=0.01 0.01 0.01; visual mesh filename=package://intro_robotics_labs/my_CAD/shoulder.stl scale=0.01 0.01 0.01
- added link lr_wheel_front, mass 1.0; collision mesh filename=package://intro_robotics_labs/my_CAD/wheel.stl scale=0.001 0.001 0.001; visual mesh filename=package://intro_robotics_labs/my_CAD/wheel.stl scale=0.001 0.001 0.001
- added link lr_wheel_rear, mass 1.0; collision mesh filename=package://intro_robotics_labs/my_CAD/wheel.stl scale=0.001 0.001 0.001; visual mesh filename=package://intro_robotics_labs/my_CAD/wheel.stl scale=0.001 0.001 0.001
- added link rf_foot, mass 1.0; collision cylinder length=0.1 radius=0.015; visual cylinder length=0.1 radius=0.001
- added link rf_foot_mid, mass 1.0; collision cylinder length=0.025 radius=0.001; visual cylinder length=0.025 radius=0.001
- added link rf_foot_mid_2, mass 1.0; collision sphere radius=0.005; visual sphere radius=0.005
- added link rf_foot_r, mass 1.0; collision sphere radius=0.01; visual sphere radius=0.01
- added link rf_leg, mass 1.0; collision cylinder length=0.1 radius=0.01; visual cylinder length=0.1 radius=0.0125
- added link rf_leg_ext, mass 1.0; collision cylinder length=0.1 radius=0.01; visual cylinder length=0.1 radius=0.0075
- added link rf_shoulder, mass 0.5; collision mesh filename=package://intro_robotics_labs/my_CAD/shoulder.stl scale=0.01 0.01 0.01; visual mesh filename=package://intro_robotics_labs/my_CAD/shoulder.stl scale=0.01 0.01 0.01
- added link rf_wheel_front, mass 1.0; collision mesh filename=package://intro_robotics_labs/my_CAD/wheel.stl scale=0.001 0.001 0.001; visual mesh filename=package://intro_robotics_labs/my_CAD/wheel.stl scale=0.001 0.001 0.001
- added link rf_wheel_rear, mass 1.0; collision mesh filename=package://intro_robotics_labs/my_CAD/wheel.stl scale=0.001 0.001 0.001; visual mesh filename=package://intro_robotics_labs/my_CAD/wheel.stl scale=0.001 0.001 0.001
- added link rr_foot, mass 1.0; collision cylinder length=0.1 radius=0.015; visual cylinder length=0.1 radius=0.001
- added link rr_foot_mid, mass 1.0; collision cylinder length=0.025 radius=0.001; visual cylinder length=0.025 radius=0.001
- added link rr_foot_mid_2, mass 1.0; collision sphere radius=0.005; visual sphere radius=0.005
- added link rr_foot_r, mass 1.0; collision sphere radius=0.01; visual sphere radius=0.01
- added link rr_leg, mass 1.0; collision cylinder length=0.1 radius=0.01; visual cylinder length=0.1 radius=0.0125
- added link rr_leg_ext, mass 1.0; collision cylinder length=0.1 radius=0.01; visual cylinder length=0.1 radius=0.0075
- added link rr_shoulder, mass 0.5; collision mesh filename=package://intro_robotics_labs/my_CAD/shoulder.stl scale=0.01 0.01 0.01; visual mesh filename=package://intro_robotics_labs/my_CAD/shoulder.stl scale=0.01 0.01 0.01
- added link rr_wheel_front, mass 1.0; collision mesh filename=package://intro_robotics_labs/my_CAD/wheel.stl scale=0.001 0.001 0.001; visual mesh filename=package://intro_robotics_labs/my_CAD/wheel.stl scale=0.001 0.001 0.001
- added link rr_wheel_rear, mass 1.0; collision mesh filename=package://intro_robotics_labs/my_CAD/wheel.stl scale=0.001 0.001 0.001; visual mesh filename=package://intro_robotics_labs/my_CAD/wheel.stl scale=0.001 0.001 0.001
- link base_link: mass None -> 1.0; geometry collision mesh filename=package://intro_robotics_labs/my_CAD/chassis-Body.stl scale=0.01 0.01 0.01; visual mesh filename=package://intro_robotics_labs/my_CAD/chassis-Body.stl scale=0.01 0.01 0.01
Joints:
- added joint lf_foot_joint_mid: type fixed, parent lf_foot_r, child lf_foot_mid, origin xyz=0 0 0 rpy=0 1.5707963267948966 0
- added joint lf_foot_joint_mid_2: type fixed, parent lf_foot_mid, child lf_foot_mid_2, origin xyz=0.025 0 0 rpy=0 -1.5707963267948966 0
- added joint lf_foot_joint_pitch: type revolute, parent lf_leg_ext, child lf_foot_r, origin xyz=0.155 0 0 rpy=0 0 1.5707963267948966, axis 0 0 1, limit lower=-1.0471975511965976 upper=1.0471975511965976 effort=100 velocity=1.0
- added joint lf_foot_joint_roll: type revolute, parent lf_foot_mid_2, child lf_foot, origin xyz=0 0 0, axis 1 0 0, limit lower=-0.39269908169872414 upper=0.39269908169872414 effort=100 velocity=1.0
- added joint lf_shoulder1_joint: type revolute, parent base_link, child lf_shoulder, origin xyz=-0.075 0.125 0 rpy=0 1.5707963267948966 0, axis 0 0 1, limit lower=-1.5707963267948966 upper=1.5707963267948966 effort=100 velocity=1.0
- added joint lf_shoulder2_joint: type fixed, parent lf_shoulder, child lf_leg, origin xyz=0 0 0
- added joint lf_suspention_ext_joint: type prismatic, parent lf_leg, child lf_leg_ext, origin xyz=0 0 0, axis 1 0 0, limit lower=0.0 upper=0.075 effort=100 velocity=10
- added joint lf_wheel_front_joint: type revolute, parent lf_foot, child lf_wheel_front, origin xyz=0.105 0 0, axis 0 0 1, limit lower=-100 upper=100 effort=100 velocity=1.0
- added joint lf_wheel_rear_joint: type revolute, parent lf_foot, child lf_wheel_rear, origin xyz=0 0.0 0, axis 0 0 1, limit lower=-100 upper=100 effort=100 velocity=1.0
- added joint lr_foot_joint_mid: type fixed, parent lr_foot_r, child lr_foot_mid, origin xyz=0 0 0 rpy=0 1.5707963267948966 0
- added joint lr_foot_joint_mid_2: type fixed, parent lr_foot_mid, child lr_foot_mid_2, origin xyz=0.025 0 0 rpy=0 -1.5707963267948966 0
- added joint lr_foot_joint_pitch: type revolute, parent lr_leg_ext, child lr_foot_r, origin xyz=0.155 0 0 rpy=0 0 1.5707963267948966, axis 0 0 1, limit lower=-1.0471975511965976 upper=1.0471975511965976 effort=100 velocity=1.0
- added joint lr_foot_joint_roll: type revolute, parent lr_foot_mid_2, child lr_foot, origin xyz=0 0 0, axis 1 0 0, limit lower=-0.39269908169872414 upper=0.39269908169872414 effort=100 velocity=1.0
- added joint lr_shoulder1_joint: type revolute, parent base_link, child lr_shoulder, origin xyz=-0.075 -0.125 0 rpy=0 1.5707963267948966 0, axis 0 0 1, limit lower=-1.5707963267948966 upper=1.5707963267948966 effort=100 velocity=1.0
- added joint lr_shoulder2_joint: type fixed, parent lr_shoulder, child lr_leg, origin xyz=0 0 0
- added joint lr_suspention_ext_joint: type prismatic, parent lr_leg, child lr_leg_ext, origin xyz=0 0 0, axis 1 0 0, limit lower=0.0 upper=0.075 effort=100 velocity=10
- added joint lr_wheel_front_joint: type revolute, parent lr_foot, child lr_wheel_front, origin xyz=0.105 0 0, axis 0 0 1, limit lower=-100 upper=100 effort=100 velocity=1.0
- added joint lr_wheel_rear_joint: type revolute, parent lr_foot, child lr_wheel_rear, origin xyz=0 0.0 0, axis 0 0 1, limit lower=-100 upper=100 effort=100 velocity=1.0
- added joint rf_foot_joint_mid: type fixed, parent rf_foot_r, child rf_foot_mid, origin xyz=0 0 0 rpy=0 1.5707963267948966 0
- added joint rf_foot_joint_mid_2: type fixed, parent rf_foot_mid, child rf_foot_mid_2, origin xyz=-0.025 0 0 rpy=0 -1.5707963267948966 0
- added joint rf_foot_joint_pitch: type revolute, parent rf_leg_ext, child rf_foot_r, origin xyz=0.155 0 0 rpy=0 0 1.5707963267948966, axis 0 0 1, limit lower=-1.0471975511965976 upper=1.0471975511965976 effort=100 velocity=1.0
- added joint rf_foot_joint_roll: type revolute, parent rf_foot_mid_2, child rf_foot, origin xyz=0 0 0, axis 1 0 0, limit lower=-0.39269908169872414 upper=0.39269908169872414 effort=100 velocity=1.0
- added joint rf_shoulder1_joint: type revolute, parent base_link, child rf_shoulder, origin xyz=0.075 0.125 0 rpy=0 1.5707963267948966 0, axis 0 0 1, limit lower=-1.5707963267948966 upper=1.5707963267948966 effort=100 velocity=1.0
- added joint rf_shoulder2_joint: type fixed, parent rf_shoulder, child rf_leg, origin xyz=0 0 0
- added joint rf_suspention_ext_joint: type prismatic, parent rf_leg, child rf_leg_ext, origin xyz=0 0 0, axis 1 0 0, limit lower=0.0 upper=0.075 effort=100 velocity=10
- added joint rf_wheel_front_joint: type revolute, parent rf_foot, child rf_wheel_front, origin xyz=0.105 0 0, axis 0 0 1, limit lower=-100 upper=100 effort=100 velocity=1.0
- added joint rf_wheel_rear_joint: type revolute, parent rf_foot, child rf_wheel_rear, origin xyz=0 0.0 0, axis 0 0 1, limit lower=-100 upper=100 effort=100 velocity=1.0
- added joint rr_foot_joint_mid: type fixed, parent rr_foot_r, child rr_foot_mid, origin xyz=0 0 0 rpy=0 1.5707963267948966 0
- added joint rr_foot_joint_mid_2: type fixed, parent rr_foot_mid, child rr_foot_mid_2, origin xyz=-0.025 0 0 rpy=0 -1.5707963267948966 0
- added joint rr_foot_joint_pitch: type revolute, parent rr_leg_ext, child rr_foot_r, origin xyz=0.155 0 0 rpy=0 0 1.5707963267948966, axis 0 0 1, limit lower=-1.0471975511965976 upper=1.0471975511965976 effort=100 velocity=1.0
- added joint rr_foot_joint_roll: type revolute, parent rr_foot_mid_2, child rr_foot, origin xyz=0 0 0, axis 1 0 0, limit lower=-0.39269908169872414 upper=0.39269908169872414 effort=100 velocity=1.0
- added joint rr_shoulder1_joint: type revolute, parent base_link, child rr_shoulder, origin xyz=0.075 -0.125 0 rpy=0 1.5707963267948966 0, axis 0 0 1, limit lower=-1.5707963267948966 upper=1.5707963267948966 effort=100 velocity=1.0
- added joint rr_shoulder2_joint: type fixed, parent rr_shoulder, child rr_leg, origin xyz=0 0 0
- added joint rr_suspention_ext_joint: type prismatic, parent rr_leg, child rr_leg_ext, origin xyz=0 0 0, axis 1 0 0, limit lower=0.0 upper=0.075 effort=100 velocity=10
- added joint rr_wheel_front_joint: type revolute, parent rr_foot, child rr_wheel_front, origin xyz=0.105 0 0, axis 0 0 1, limit lower=-100 upper=100 effort=100 velocity=1.0
- added joint rr_wheel_rear_joint: type revolute, parent rr_foot, child rr_wheel_rear, origin xyz=0 0.0 0, axis 0 0 1, limit lower=-100 upper=100 effort=100 velocity=1.0

Commit message: FIX Package rename

File: urdf/HEBI.urdf (robot description, URDF)
Before this commit: robot simple_robot, 38 links, 37 joints
Links:
- link base_link: geometry collision mesh filename=package://hebi_robot/my_CAD/chassis-Body.stl scale=0.01 0.01 0.01; visual mesh filename=package://hebi_robot/my_CAD/chassis-Body.stl scale=0.01 0.01 0.01
- link lf_shoulder: geometry collision mesh filename=package://hebi_robot/my_CAD/shoulder.stl scale=0.01 0.01 0.01; visual mesh filename=package://hebi_robot/my_CAD/shoulder.stl scale=0.01 0.01 0.01
- link lf_wheel_front: geometry collision mesh filename=package://hebi_robot/my_CAD/wheel.stl scale=0.001 0.001 0.001; visual mesh filename=package://hebi_robot/my_CAD/wheel.stl scale=0.001 0.001 0.001
- link lf_wheel_rear: geometry collision mesh filename=package://hebi_robot/my_CAD/wheel.stl scale=0.001 0.001 0.001; visual mesh filename=package://hebi_robot/my_CAD/wheel.stl scale=0.001 0.001 0.001
- link lr_shoulder: geometry collision mesh filename=package://hebi_robot/my_CAD/shoulder.stl scale=0.01 0.01 0.01; visual mesh filename=package://hebi_robot/my_CAD/shoulder.stl scale=0.01 0.01 0.01
- link lr_wheel_front: geometry collision mesh filename=package://hebi_robot/my_CAD/wheel.stl scale=0.001 0.001 0.001; visual mesh filename=package://hebi_robot/my_CAD/wheel.stl scale=0.001 0.001 0.001
- link lr_wheel_rear: geometry collision mesh filename=package://hebi_robot/my_CAD/wheel.stl scale=0.001 0.001 0.001; visual mesh filename=package://hebi_robot/my_CAD/wheel.stl scale=0.001 0.001 0.001
- link rf_shoulder: geometry collision mesh filename=package://hebi_robot/my_CAD/shoulder.stl scale=0.01 0.01 0.01; visual mesh filename=package://hebi_robot/my_CAD/shoulder.stl scale=0.01 0.01 0.01
- link rf_wheel_front: geometry collision mesh filename=package://hebi_robot/my_CAD/wheel.stl scale=0.001 0.001 0.001; visual mesh filename=package://hebi_robot/my_CAD/wheel.stl scale=0.001 0.001 0.001
- link rf_wheel_rear: geometry collision mesh filename=package://hebi_robot/my_CAD/wheel.stl scale=0.001 0.001 0.001; visual mesh filename=package://hebi_robot/my_CAD/wheel.stl scale=0.001 0.001 0.001
- link rr_shoulder: geometry collision mesh filename=package://hebi_robot/my_CAD/shoulder.stl scale=0.01 0.01 0.01; visual mesh filename=package://hebi_robot/my_CAD/shoulder.stl scale=0.01 0.01 0.01
- link rr_wheel_front: geometry collision mesh filename=package://hebi_robot/my_CAD/wheel.stl scale=0.001 0.001 0.001; visual mesh filename=package://hebi_robot/my_CAD/wheel.stl scale=0.001 0.001 0.001
- link rr_wheel_rear: geometry collision mesh filename=package://hebi_robot/my_CAD/wheel.stl scale=0.001 0.001 0.001; visual mesh filename=package://hebi_robot/my_CAD/wheel.stl scale=0.001 0.001 0.001

File: urdf/HEBI.urdf.xacro (robot description, xacro)
@@ -13,5 +13,5 @@
     <visual>
       <geometry>
-        <mesh filename="package://intro_robotics_labs/my_CAD/chassis-Body.stl" scale="0.01 0.01 0.01"/>
+        <mesh filename="package://hebi_robot/my_CAD/chassis-Body.stl" scale="0.01 0.01 0.01"/>
       </geometry>
       <origin xyz="0 0 0" rpy="0 0 0"/>
@@ -20,5 +20,5 @@
     <collision>
       <geometry>
-        <mesh filename="package://intro_robotics_labs/my_CAD/chassis-Body.stl" scale="0.01 0.01 0.01"/>
+        <mesh filename="package://hebi_robot/my_CAD/chassis-Body.stl" scale="0.01 0.01 0.01"/>
       </geometry>
       <origin xyz="0 0 0" rpy="0 0 0"/>
@@ -45,5 +45,5 @@
       <visual>
         <geometry>
-          <mesh filename="package://intro_robotics_labs/my_CAD/shoulder.stl" scale="0.01 0.01 0.01"/>
+          <mesh filename="package://hebi_robot/my_CAD/shoulder.stl" scale="0.01 0.01 0.01"/>
         </geometry>
         <origin xyz="0 0 0" rpy="${-pi/2} 0 ${pi/2}"/>
@@ -52,5 +52,5 @@
       <collision>
         <geometry>
-          <mesh filename="package://intro_robotics_labs/my_CAD/shoulder.stl" scale="0.01 0.01 0.01"/>
+          <mesh filename="package://hebi_robot/my_CAD/shoulder.stl" scale="0.01 0.01 0.01"/>
         </geometry>
       </collision>
@@ -236,5 +236,5 @@
       <visual>
         <geometry>
-          <mesh filename="package://intro_robotics_labs/my_CAD/wheel.stl" scale="0.001 0.001 0.001"/>
+          <mesh filename="package://hebi_robot/my_CAD/wheel.stl" scale="0.001 0.001 0.001"/>
         </geometry>
         <origin xyz="0 0 0" rpy="${-pi/2} ${pi/2} 0"/>
@@ -243,5 +243,5 @@
       <collision>
         <geometry>
-          <mesh filename="package://intro_robotics_labs/my_CAD/wheel.stl" scale="0.001 0.001 0.001"/>
+          <mesh filename="package://hebi_robot/my_CAD/wheel.stl" scale="0.001 0.001 0.001"/>
         </geometry>
         <origin xyz="0 0 0"/>
@@ -265,5 +265,5 @@
       <visual>
         <geometry>
-          <mesh filename="package://intro_robotics_labs/my_CAD/wheel.stl" scale="0.001 0.001 0.001"/>
+          <mesh filename="package://hebi_robot/my_CAD/wheel.stl" scale="0.001 0.001 0.001"/>
         </geometry>
           <origin xyz="0 0 0" rpy="${-pi/2} ${pi/2} 0"/>
@@ -272,5 +272,5 @@
       <collision>
         <geometry>
-          <mesh filename="package://intro_robotics_labs/my_CAD/wheel.stl" scale="0.001 0.001 0.001"/>
+          <mesh filename="package://hebi_robot/my_CAD/wheel.stl" scale="0.001 0.001 0.001"/>
         </geometry>
         <origin xyz="0 0 0"/>
@@ -297,5 +297,5 @@
       <visual>
         <geometry>
-          <mesh filename="package://intro_robotics_labs/my_CAD/shoulder.stl" scale="0.01 0.01 0.01"/>
+          <mesh filename="package://hebi_robot/my_CAD/shoulder.stl" scale="0.01 0.01 0.01"/>
         </geometry>
         <origin xyz="0 0 0" rpy="${-pi/2} 0 ${pi/2}"/>
@@ -304,5 +304,5 @@
       <collision>
         <geometry>
-          <mesh filename="package://intro_robotics_labs/my_CAD/shoulder.stl" scale="0.01 0.01 0.01"/>
+          <mesh filename="package://hebi_robot/my_CAD/shoulder.stl" scale="0.01 0.01 0.01"/>
         </geometry>
       </collision>
@@ -488,5 +488,5 @@
       <visual>
         <geometry>
-          <mesh filename="package://intro_robotics_labs/my_CAD/wheel.stl" scale="0.001 0.001 0.001"/>
+          <mesh filename="package://hebi_robot/my_CAD/wheel.stl" scale="0.001 0.001 0.001"/>
         </geometry>
         <origin xyz="0 0 0" rpy="${-pi/2} ${-pi/2} 0"/>
@@ -495,5 +495,5 @@
       <collision>
         <geometry>
-          <mesh filename="package://intro_robotics_labs/my_CAD/wheel.stl" scale="0.001 0.001 0.001"/>
+          <mesh filename="package://hebi_robot/my_CAD/wheel.stl" scale="0.001 0.001 0.001"/>
         </geometry>
         <origin xyz="0 0 0"/>
@@ -517,5 +517,5 @@
       <visual>
         <geometry>
-          <mesh filename="package://intro_robotics_labs/my_CAD/wheel.stl" scale="0.001 0.001 0.001"/>
+          <mesh filename="package://hebi_robot/my_CAD/wheel.stl" scale="0.001 0.001 0.001"/>
         </geometry>
           <origin xyz="0 0 0" rpy="${-pi/2} ${-pi/2} 0"/>
@@ -524,5 +524,5 @@
       <collision>
         <geometry>
-          <mesh filename="package://intro_robotics_labs/my_CAD/wheel.stl" scale="0.001 0.001 0.001"/>
+          <mesh filename="package://hebi_robot/my_CAD/wheel.stl" scale="0.001 0.001 0.001"/>
         </geometry>
         <origin xyz="0 0 0"/>

Commit message: robot moves good

File: urdf/HEBI.urdf (robot description, URDF)
Before this commit: robot HEBI, 38 links, 37 joints
Joints:
- joint rf_shoulder1_joint: limit lower=-1.5707963267948966 upper=1.5707963267948966 effort=100 velocity=1.0 -> lower=-1.5707963267948966 upper=1.5707963267948966 effort=100 velocity=10.0
- joint rf_suspention_ext_joint: limit lower=0.0 upper=0.075 effort=100 velocity=10 -> lower=0.0 upper=0.075 effort=100 velocity=1
