Commit message: UPDATE Naming

File: urdf/HEBI.urdf.xacro (robot description, xacro)
@@ -4,4 +4,5 @@
   <xacro:property name="pi" value="3.141592653589793"/>
   <!-- Base -->
+  <!--
   <link name="world"/>
   <joint name="world_joint" type="fixed">
@@ -10,8 +11,9 @@
     <origin rpy="0.0 0.0 0.0" xyz="0.0 0.0 0.0"/>
   </joint>
+  -->
   <link name="base_link">
     <visual>
       <geometry>
-        <mesh filename="package://hebi_robot/my_CAD/chassis-Body.stl" scale="0.01 0.01 0.01"/>
+        <mesh filename="package://hebi_robot/meshes/chassis-Body.stl" scale="0.01 0.01 0.01"/>
       </geometry>
       <origin xyz="0 0 0" rpy="0 0 0"/>
@@ -20,5 +22,5 @@
     <collision>
       <geometry>
-        <mesh filename="package://hebi_robot/my_CAD/chassis-Body.stl" scale="0.01 0.01 0.01"/>
+        <mesh filename="package://hebi_robot/meshes/chassis-Body.stl" scale="0.01 0.01 0.01"/>
       </geometry>
       <origin xyz="0 0 0" rpy="0 0 0"/>
@@ -45,5 +47,5 @@
       <visual>
         <geometry>
-          <mesh filename="package://hebi_robot/my_CAD/shoulder.stl" scale="0.01 0.01 0.01"/>
+          <mesh filename="package://hebi_robot/meshes/shoulder.stl" scale="0.01 0.01 0.01"/>
         </geometry>
         <origin xyz="0 0 0" rpy="${-pi/2} 0 ${pi/2}"/>
@@ -52,5 +54,5 @@
       <collision>
         <geometry>
-          <mesh filename="package://hebi_robot/my_CAD/shoulder.stl" scale="0.01 0.01 0.01"/>
+          <mesh filename="package://hebi_robot/meshes/shoulder.stl" scale="0.01 0.01 0.01"/>
         </geometry>
       </collision>
@@ -236,5 +238,5 @@
       <visual>
         <geometry>
-          <mesh filename="package://hebi_robot/my_CAD/wheel.stl" scale="0.001 0.001 0.001"/>
+          <mesh filename="package://hebi_robot/meshes/wheel.stl" scale="0.001 0.001 0.001"/>
         </geometry>
         <origin xyz="0 0 0" rpy="${-pi/2} ${pi/2} 0"/>
@@ -243,5 +245,5 @@
       <collision>
         <geometry>
-          <mesh filename="package://hebi_robot/my_CAD/wheel.stl" scale="0.001 0.001 0.001"/>
+          <mesh filename="package://hebi_robot/meshes/wheel.stl" scale="0.001 0.001 0.001"/>
         </geometry>
         <origin xyz="0 0 0"/>
@@ -265,5 +267,5 @@
       <visual>
         <geometry>
-          <mesh filename="package://hebi_robot/my_CAD/wheel.stl" scale="0.001 0.001 0.001"/>
+          <mesh filename="package://hebi_robot/meshes/wheel.stl" scale="0.001 0.001 0.001"/>
         </geometry>
           <origin xyz="0 0 0" rpy="${-pi/2} ${pi/2} 0"/>
@@ -272,5 +274,5 @@
       <collision>
         <geometry>
-          <mesh filename="package://hebi_robot/my_CAD/wheel.stl" scale="0.001 0.001 0.001"/>
+          <mesh filename="package://hebi_robot/meshes/wheel.stl" scale="0.001 0.001 0.001"/>
         </geometry>
         <origin xyz="0 0 0"/>
@@ -297,5 +299,5 @@
       <visual>
         <geometry>
-          <mesh filename="package://hebi_robot/my_CAD/shoulder.stl" scale="0.01 0.01 0.01"/>
+          <mesh filename="package://hebi_robot/meshes/shoulder.stl" scale="0.01 0.01 0.01"/>
         </geometry>
         <origin xyz="0 0 0" rpy="${-pi/2} 0 ${pi/2}"/>
@@ -304,5 +306,5 @@
       <collision>
         <geometry>
-          <mesh filename="package://hebi_robot/my_CAD/shoulder.stl" scale="0.01 0.01 0.01"/>
+          <mesh filename="package://hebi_robot/meshes/shoulder.stl" scale="0.01 0.01 0.01"/>
         </geometry>
       </collision>
@@ -488,5 +490,5 @@
       <visual>
         <geometry>
-          <mesh filename="package://hebi_robot/my_CAD/wheel.stl" scale="0.001 0.001 0.001"/>
+          <mesh filename="package://hebi_robot/meshes/wheel.stl" scale="0.001 0.001 0.001"/>
         </geometry>
         <origin xyz="0 0 0" rpy="${-pi/2} ${-pi/2} 0"/>
@@ -495,5 +497,5 @@
       <collision>
         <geometry>
-          <mesh filename="package://hebi_robot/my_CAD/wheel.stl" scale="0.001 0.001 0.001"/>
+          <mesh filename="package://hebi_robot/meshes/wheel.stl" scale="0.001 0.001 0.001"/>
         </geometry>
         <origin xyz="0 0 0"/>
@@ -517,5 +519,5 @@
       <visual>
         <geometry>
-          <mesh filename="package://hebi_robot/my_CAD/wheel.stl" scale="0.001 0.001 0.001"/>
+          <mesh filename="package://hebi_robot/meshes/wheel.stl" scale="0.001 0.001 0.001"/>
         </geometry>
           <origin xyz="0 0 0" rpy="${-pi/2} ${-pi/2} 0"/>
@@ -524,5 +526,5 @@
       <collision>
         <geometry>
-          <mesh filename="package://hebi_robot/my_CAD/wheel.stl" scale="0.001 0.001 0.001"/>
+          <mesh filename="package://hebi_robot/meshes/wheel.stl" scale="0.001 0.001 0.001"/>
         </geometry>
         <origin xyz="0 0 0"/>

File: urdf/hebi.urdf (robot description, URDF)
Before this commit: robot HEBI, 2 links, 1 joints
Links:
- link base_link: geometry collision mesh filename=package://hebi_robot/meshes/chassis-Body.stl scale=0.01 0.01 0.01; visual mesh filename=package://hebi_robot/meshes/chassis-Body.stl scale=0.01 0.01 0.01

Commit message: ADD Transmissions to xarco

File: urdf/HEBI.urdf.xacro (robot description, xacro)
@@ -44,4 +44,11 @@
       <dynamics damping="0.5" friction="0.2"/>
     </joint>
+    <transmission name="{left}_shoulder1_trans">
+      <type>transmission_interface/SimpleTransmission</type>
+      <joint name="{left}_shoulder1_joint">
+        <hardwareInterface>EffortJointInterface</hardwareInterface>
+      </joint>
+      <actuator name="{left}_shoulder1_motor"/>
+    </transmission>
     <link name="${left}_shoulder">
       <visual>
@@ -125,4 +132,11 @@
       <dynamics damping="0.1" friction="0.1"/>
     </joint>
+    <transmission name="{left}_foot_joint_pitch_trans">
+      <type>transmission_interface/SimpleTransmission</type>
+      <joint name="{left}_foot_joint_pitch">
+        <hardwareInterface>EffortJointInterface</hardwareInterface>
+      </joint>
+      <actuator name="{left}_foot_joint_pitch_motor"/>
+    </transmission>
     <link name="${left}_foot_r">
       <visual>
@@ -206,4 +220,11 @@
       <dynamics damping="0.1" friction="0.1"/>
     </joint>
+    <transmission name="{left}_foot_joint_roll_trans">
+      <type>transmission_interface/SimpleTransmission</type>
+      <joint name="{left}_foot_joint_roll">
+        <hardwareInterface>EffortJointInterface</hardwareInterface>
+      </joint>
+      <actuator name="{left}_foot_joint_roll_motor"/>
+    </transmission>
     <link name="${left}_foot">
       <visual>
@@ -234,4 +255,6 @@
       <limit lower="${-100}" upper="${100}" effort="100" velocity="1.0"/>
       <dynamics damping="0.1" friction="0.1"/>
+      <!-- BIND TO TRASMISSION -->
+      <mimic joint="${left}_wheel_rear_joint" multiplier="1.0"/>
     </joint>
     <link name="${left}_wheel_front">
@@ -264,4 +287,11 @@
       <dynamics damping="0.1" friction="0.1"/>
     </joint>
+    <transmission name="{left}_wheel_rear_trans">
+      <type>transmission_interface/SimpleTransmission</type>
+      <joint name="{left}_wheel_rear_joint">
+        <hardwareInterface>EffortJointInterface</hardwareInterface>
+      </joint>
+      <actuator name="{left}_wheel_rear_motor"/>
+    </transmission>
     <link name="${left}_wheel_rear">
       <visual>
@@ -296,4 +326,11 @@
       <dynamics damping="0.5" friction="0.2"/>
     </joint>
+    <transmission name="{right}_shoulder1_trans">
+      <type>transmission_interface/SimpleTransmission</type>
+      <joint name="{right}_shoulder1_joint">
+        <hardwareInterface>EffortJointInterface</hardwareInterface>
+      </joint>
+      <actuator name="{right}_shoulder1_motor"/>
+    </transmission>
     <link name="${right}_shoulder">
       <visual>
@@ -377,4 +414,11 @@
       <dynamics damping="0.1" friction="0.1"/>
     </joint>
+    <transmission name="{right}_foot_joint_pitch_trans">
+      <type>transmission_interface/SimpleTransmission</type>
+      <joint name="{right}_foot_joint_pitch">
+        <hardwareInterface>EffortJointInterface</hardwareInterface>
+      </joint>
+      <actuator name="{right}_foot_joint_pitch_motor"/>
+    </transmission>
     <link name="${right}_foot_r">
       <visual>
@@ -458,4 +502,11 @@
       <dynamics damping="0.1" friction="0.1"/>
     </joint>
+    <transmission name="{right}_foot_joint_roll_trans">
+      <type>transmission_interface/SimpleTransmission</type>
+      <joint name="{right}_foot_joint_roll">
+        <hardwareInterface>EffortJointInterface</hardwareInterface>
+      </joint>
+      <actuator name="{right}_foot_joint_roll_motor"/>
+    </transmission>
     <link name="${right}_foot">
       <visual>
@@ -486,4 +537,6 @@
       <limit lower="${-100}" upper="${100}" effort="100" velocity="1.0"/>
       <dynamics damping="0.1" friction="0.1"/>
+      <!-- BIND TO TRASMISSION -->
+      <mimic joint="${right}_wheel_rear_joint" multiplier="1.0"/>
     </joint>
     <link name="${right}_wheel_front">
@@ -516,4 +569,11 @@
       <dynamics damping="0.1" friction="0.1"/>
     </joint>
+    <transmission name="{right}_wheel_rear_trans">
+      <type>transmission_interface/SimpleTransmission</type>
+      <joint name="{right}_wheel_rear_joint">
+        <hardwareInterface>EffortJointInterface</hardwareInterface>
+      </joint>
+      <actuator name="{right}_wheel_rear_motor"/>
+    </transmission>
     <link name="${right}_wheel_rear">
       <visual>
